Commit message: dealing with joint4

File: robots/common/franka_arm.ros2_control.xacro (robot description, xacro)
@@ -60,5 +60,5 @@
       <xacro:configure_joint joint_name="${arm_prefix_modified}${arm_id}_joint2" initial_position="${-pi/4}"/>
       <xacro:configure_joint joint_name="${arm_prefix_modified}${arm_id}_joint3" initial_position="0.0"/>
-      <xacro:configure_joint joint_name="${arm_prefix_modified}${arm_id}_joint4" initial_position="${-3*pi/4}"/>
+      <xacro:configure_joint joint_name="${arm_prefix_modified}${arm_id}_joint4" initial_position="0.0"/>
       <xacro:configure_joint joint_name="${arm_prefix_modified}${arm_id}_joint5" initial_position="0.0"/>
       <xacro:configure_joint joint_name="${arm_prefix_modified}${arm_id}_joint6" initial_position="${pi/2}"/>

File: robots/common/franka_arm.xacro (robot description, xacro)
@@ -76,5 +76,5 @@
       <parent link="${prefix}link3" />
       <child link="${prefix}link4" />
-      <axis xyz="0 0 1" />
+      <axis xyz="0 1 0" />
       <xacro:franka-limits name="joint4" config="${joint_limits}" />
       <xacro:franka-dynamics name="joint4" config="${dynamics}" />

Commit message: fixing joint5

File: robots/common/franka_arm.ros2_control.xacro (robot description, xacro)
@@ -61,5 +61,5 @@
       <xacro:configure_joint joint_name="${arm_prefix_modified}${arm_id}_joint3" initial_position="0.0"/>
       <xacro:configure_joint joint_name="${arm_prefix_modified}${arm_id}_joint4" initial_position="${-3*pi/4}"/>
-      <xacro:configure_joint joint_name="${arm_prefix_modified}${arm_id}_joint5" initial_position="${pi/2}"/>
+      <xacro:configure_joint joint_name="${arm_prefix_modified}${arm_id}_joint5" initial_position="0.0"/>
       <xacro:configure_joint joint_name="${arm_prefix_modified}${arm_id}_joint6" initial_position="${pi/2}"/>
       <xacro:configure_joint joint_name="${arm_prefix_modified}${arm_id}_joint7" initial_position="${pi/4}"/>

File: robots/common/franka_arm.xacro (robot description, xacro)
@@ -90,5 +90,5 @@
       <parent link="${prefix}link4" />
       <child link="${prefix}link5" />
-      <axis xyz="0 0 1" />
+      <axis xyz="1 0 0" />
       <xacro:franka-limits name="joint5" config="${joint_limits}" />
       <xacro:franka-dynamics name="joint5" config="${dynamics}" />

Commit message: further work on arm with updated collada files

File: robots/common/franka_arm.ros2_control.xacro (robot description, xacro)
@@ -25,8 +25,13 @@
           </xacro:if>
           <xacro:if value="${use_fake_hardware == 0 and gazebo == 0 and multi_arm == 0}">
+            <plugin>dynamixel_hardware/DynamixelHardware</plugin>
+            <param name="usb_port">/dev/ttyACM0</param>
+            <param name="baud_rate">1000000</param>
+          </xacro:if>
+          <!-- <xacro:if value="${use_fake_hardware == 0 and gazebo == 0 and multi_arm == 0}">
             <plugin>franka_hardware/FrankaHardwareInterface</plugin>
             <param name="robot_ip">${robot_ip}</param>
             <param name="arm_prefix">${arm_prefix}</param>
-          </xacro:if>
+          </xacro:if> -->
           <xacro:if value="${use_fake_hardware == 0 and gazebo == 0 and multi_arm == 1}">
             <plugin>franka_hardware/MultiFrankaHardwareInterface</plugin>
@@ -57,11 +62,11 @@
         </joint>
       </xacro:macro>
-      <xacro:configure_joint joint_name="${arm_prefix_modified}${arm_id}_joint1" initial_position="0.0"/>
+      <xacro:configure_joint joint_name="${arm_prefix_modified}${arm_id}_joint1" initial_position="${pi}"/>
       <xacro:configure_joint joint_name="${arm_prefix_modified}${arm_id}_joint2" initial_position="0.0"/>
       <xacro:configure_joint joint_name="${arm_prefix_modified}${arm_id}_joint3" initial_position="0.0"/>
       <xacro:configure_joint joint_name="${arm_prefix_modified}${arm_id}_joint4" initial_position="0.0"/>
-      <xacro:configure_joint joint_name="${arm_prefix_modified}${arm_id}_joint5" initial_position="0.0"/>
-      <xacro:configure_joint joint_name="${arm_prefix_modified}${arm_id}_joint6" initial_position="${pi/2}"/>
-      <xacro:configure_joint joint_name="${arm_prefix_modified}${arm_id}_joint7" initial_position="${pi/4}"/>
+      <xacro:configure_joint joint_name="${arm_prefix_modified}${arm_id}_joint5" initial_position="${pi/2}"/>
+      <xacro:configure_joint joint_name="${arm_prefix_modified}${arm_id}_joint6" initial_position="${pi}"/>
+      <xacro:configure_joint joint_name="${arm_prefix_modified}${arm_id}_joint7" initial_position="0"/>
       <xacro:if value="${gazebo and hand}">
         <xacro:configure_joint joint_name="${arm_id}_finger_joint1" initial_position="0.0" />

File: robots/common/franka_arm.xacro (robot description, xacro)
@@ -90,5 +90,5 @@
       <parent link="${prefix}link4" />
       <child link="${prefix}link5" />
-      <axis xyz="1 0 0" />
+      <axis xyz="0 0 1" />
       <xacro:franka-limits name="joint5" config="${joint_limits}" />
       <xacro:franka-dynamics name="joint5" config="${dynamics}" />
@@ -117,5 +117,5 @@
       <parent link="${prefix}link6"/>
       <child link="${prefix}link7"/>
-      <axis xyz="0 0 1"/>
+      <axis xyz="1 0 0"/>
       <xacro:franka-limits name="joint7" config="${joint_limits}" />
       <xacro:franka-dynamics name="joint7" config="${dynamics}" />
